Commit message: working odometry

File: description/gazebo_control.xacro (robot description, xacro)
@@ -13,5 +13,5 @@
             <!-- Output -->
             <odometry_frame>odom</odometry_frame>
-            <robot_base_frame>base_link</robot_base_frame>
+            <robot_base_frame>base_footprint</robot_base_frame>
             <publish_odom>true</publish_odom>
             <publish_odom_tf>true</publish_odom_tf>

File: description/robot.urdf.xacro (robot description, xacro)
@@ -4,3 +4,7 @@
     <xacro:include filename="gazebo_control.xacro" />
     <xacro:include filename="lidar.xacro" />
+    <!-- <xacro:laser_bug parent="world">
+    <origin xyz="0 0 0" rpy="0 0 0" />
+  </xacro:laser_bug> -->
+  <!-- <xacro:mx_ros_2_control name="mx_ros_2_control" /> -->
 </robot>

File: description/robot_core.xacro (robot description, xacro)
@@ -14,6 +14,18 @@
         <color rgba="0 0 0 1"/>
     </material>
+      <!-- ROBOT BASE FOOTPRINT -->
+    <!-- Define the center of the main robot chassis projected on the ground -->
+    <!-- <link name="base_footprint" > </link> -->
+    <!-- The base footprint of the robot is located underneath the chassis -->
+    <!-- <joint name="base_joint" type="fixed">
+        <parent link="base_footprint"/>
+        <child link="base_link" />
+        <origin xyz="0.0 0.0 0.02" rpy="0 0 0"/>
+    </joint> -->
     <!-- BASE LINK -->
     <link name="base_link">
+        <!-- <visual>
+            <origin xyz="0.0 0.0 0.0"/>
+        </visual> -->
     </link>
     <!-- CHASSIS LINK -->

File: description/ros2_control.xacro (robot description, xacro)
@@ -22,8 +22,8 @@
         </joint>
     </ros2_control>
-    <gazebo>
+    <!-- <gazebo>
         <plugin name="gazebo_ros2_control" filename="libgazebo_ros2_control.so"  >
             <parameters>$(find laser_bug)/config/my_controllers.yaml</parameters>
         </plugin>
-    </gazebo>
+    </gazebo> -->
 </robot>
